Commit message: 2025/4/1_final

File: src/tjurm_arm_final/urdf/tjurm_arm_final.urdf (robot description, URDF)
Before this commit: robot tjurm_arm_final, 8 links, 7 joints
Joints:
- joint joint1: limit lower=-3.14 upper=3.14 effort=100 velocity=1 -> lower=-1.5 upper=1.5 effort=100 velocity=1
- joint joint2: limit lower=-3.14 upper=3.14 effort=100 velocity=1 -> lower=-1.59 upper=1.2065 effort=100 velocity=1
- joint joint3: limit lower=-3.14 upper=3.14 effort=100 velocity=1 -> lower=-1.18 upper=1.62 effort=100 velocity=1
- joint joint4: limit lower=-3.14 upper=3.14 effort=100 velocity=1 -> lower=-1.9 upper=2.3 effort=100 velocity=1
- joint joint5: limit lower=-3.14 upper=3.14 effort=100 velocity=1 -> lower=-1.73 upper=1.40 effort=100 velocity=1

Commit message: update

File: src/tjurm_arm_final/urdf/tjurm_arm_final.urdf (robot description, URDF)
Before this commit: robot tjurm_arm_final, 8 links, 7 joints
Joints:
- joint fixed: origin xyz=0 0 0.1 rpy=0 0 0 -> xyz=0 0 0.255 rpy=0 0 0
